File: kicad/lab-04.sch (KiCad schematic (older format))
At the start: 18 parts, among them M1 Multimeter, M2 Multimeter

Commit message: Uppdatera kopplingsscheman.
Parts:
- added C1 (x3): 100n, symbol C
- added M1: OSCILLOSCOPE, symbol OSCILLOSCOPE
- added R1 (x2): 50, symbol R
- added R1, R2 (x3): 1k, symbol R
- added R3 (x3): 1M, symbol R
- added V1, V? (x2): Signalgenerator, symbol VACSOURCE
- R1: value 1k -> 50
Connections:
- wire segments 51 -> 102
- no-connect marks 0 -> 1
Other:
- note added: "Oscilloskop"
- note added: "SKÅPPROB"
- moved on the sheet: C1, C2, D1, L1, M1, M2, R1, R2, V1
